File: Kicad/MZ-1500_SD+NRF.kicad_pcb (KiCad board)
At the start: 2 copper layers, 114.8 x 104.4 mm, 20 parts, among them J1 MZ-1500 BUS, J2 Micro_SD_Card_Kit, J3 MicroSD Card Adapter, J4 RP2350B Left, J5 RP2350B Right, J6 VGA, U1 74LS04, U2 74LS30, U3 8255, U4 Arduino_Pro_Mini

Commit message: Add files via upload
Parts:
- added D1: BAT54, Diode_THT:D_DO-41_SOD81_P10.16mm_Horizontal, F.Cu at (174.9, 123.4)
Connections:
- J4 pad 1: +5V -> (no net)
- J4 pad 16: (no net) -> Net-(D1-Pad1)
Routing:
- net +5V: track 248.2 -> 239.7 mm
- net Net-(D1-Pad1): track 0.00 -> 7.04 mm
Other:
- board text added: "1N5819"
- board text added: "MZ-1500_SD+NiseRamFile Rev1.1"
- board text removed: "MZ-1500_SD+NiseRamFile Rev1.0"
